File: Makech/hardware/KiCad files/Makech.sch (KiCad schematic (older format))
At the start: 67 parts, among them IC1 ULN2803, J1 USB_B_Micro, J2 SWD programmer, J3 ESP32-Exp, SW1 RST, U1 CONN_01X04, U6 AP2114_3.3v, X1 Screw_Terminal_1x02

Commit message: SPI for ESP32
Parts:
- C1, C5, C6: symbol Makech-rescue:C_Small-Device-Makech-rescue-Makech-rescue-Makech-rescue -> Makech-rescue:C_Small-Device-Makech-rescue-Makech-rescue-Makech-rescue-Makech-rescue
- C2, C2.1, C3, C3.1, C4, C4.1: symbol Makech-rescue:C-RESCUE-Ogaki--Ogaki-rescue-Makech-rescue-Makech-rescue-Makech-rescue-Makech-rescue -> Makech-rescue:C-RESCUE-Ogaki--Ogaki-rescue-Makech-rescue-Makech-rescue-Makech-rescue-Makech-rescue-Makech-rescue
- D1, D1.1: symbol Makech-rescue:ZENER--Ogaki-rescue-Makech-rescue-Makech-rescue-Makech-rescue-Makech-rescue -> Makech-rescue:ZENER--Ogaki-rescue-Makech-rescue-Makech-rescue-Makech-rescue-Makech-rescue-Makech-rescue
- D2, D3: symbol Makech-rescue:D_Schottky-Device-Makech-rescue-Makech-rescue-Makech-rescue -> Makech-rescue:D_Schottky-Device-Makech-rescue-Makech-rescue-Makech-rescue-Makech-rescue
- F1, F1.1: symbol Makech-rescue:FUSE--Ogaki-rescue-Makech-rescue-Makech-rescue-Makech-rescue-Makech-rescue -> Makech-rescue:FUSE--Ogaki-rescue-Makech-rescue-Makech-rescue-Makech-rescue-Makech-rescue-Makech-rescue
- F2: symbol Makech-rescue:Fuse-Device-Makech-rescue-Makech-rescue-Makech-rescue -> Makech-rescue:Fuse-Device-Makech-rescue-Makech-rescue-Makech-rescue-Makech-rescue
- IC1: symbol Makech-rescue:ULN2803--Ogaki-rescue-Makech-rescue-Makech-rescue-Makech-rescue-Makech-rescue -> Makech-rescue:ULN2803--Ogaki-rescue-Makech-rescue-Makech-rescue-Makech-rescue-Makech-rescue-Makech-rescue
- J1: symbol Makech-rescue:USB_B_Micro-Connector-Makech-rescue-Makech-rescue-Makech-rescue -> Makech-rescue:USB_B_Micro-Connector-Makech-rescue-Makech-rescue-Makech-rescue-Makech-rescue
- J2: symbol Makech-rescue:Conn_02x02_Counter_Clockwise-Connector_Generic-Makech-rescue-Makech-rescue-Makech-rescue -> Makech-rescue:Conn_02x02_Counter_Clockwise-Connector_Generic-Makech-rescue-Makech-rescue-Makech-rescue-Makech-rescue
- JP1, JP2: symbol Makech-rescue:CONN_01X02--Ogaki-rescue-Makech-rescue-Makech-rescue-Makech-rescue-Makech-rescue -> Makech-rescue:CONN_01X02--Ogaki-rescue-Makech-rescue-Makech-rescue-Makech-rescue-Makech-rescue-Makech-rescue
- LED1, LED1.1, LED2, LED2.1, LED3, LED3.1, LED4, LED4.1: symbol Makech-rescue:LED-RESCUE-Ogaki--Ogaki-rescue-Makech-rescue-Makech-rescue-Makech-rescue-Makech-rescue -> Makech-rescue:LED-RESCUE-Ogaki--Ogaki-rescue-Makech-rescue-Makech-rescue-Makech-rescue-Makech-rescue-Makech-rescue
- R1, R2, R3, R4, R5: symbol Makech-rescue:R-SIL_8NB--Ogaki-rescue-Makech-rescue-Makech-rescue-Makech-rescue-Makech-rescue -> Makech-rescue:R-SIL_8NB--Ogaki-rescue-Makech-rescue-Makech-rescue-Makech-rescue-Makech-rescue-Makech-rescue
- R1.1, R10.1, R2.2, R3.1, R4.1, R5.1, R6.1, R7.1, R8.1, R9.1: symbol Makech-rescue:R-RESCUE-Ogaki--Ogaki-rescue-Makech-rescue-Makech-rescue-Makech-rescue-Makech-rescue -> Makech-rescue:R-RESCUE-Ogaki--Ogaki-rescue-Makech-rescue-Makech-rescue-Makech-rescue-Makech-rescue-Makech-rescue
- S1, S1.1, S2, S2.1, S3, S3.1, S4, S4.1, S5, S5.1, S7: symbol Makech-rescue:switch--Ogaki-rescue-Makech-rescue-Makech-rescue-Makech-rescue-Makech-rescue -> Makech-rescue:switch--Ogaki-rescue-Makech-rescue-Makech-rescue-Makech-rescue-Makech-rescue-Makech-rescue
- SJ2: symbol Makech-rescue:JUMPER--Ogaki-rescue-Makech-rescue-Makech-rescue-Makech-rescue-Makech-rescue -> Makech-rescue:JUMPER--Ogaki-rescue-Makech-rescue-Makech-rescue-Makech-rescue-Makech-rescue-Makech-rescue
- SW1: symbol Makech-rescue:SW_Push-Switch-Makech-rescue-Makech-rescue-Makech-rescue -> Makech-rescue:SW_Push-Switch-Makech-rescue-Makech-rescue-Makech-rescue-Makech-rescue
- U1: symbol Makech-rescue:CONN_01X04--Ogaki-rescue-Makech-rescue-Makech-rescue-Makech-rescue-Makech-rescue -> Makech-rescue:CONN_01X04--Ogaki-rescue-Makech-rescue-Makech-rescue-Makech-rescue-Makech-rescue-Makech-rescue
- U6: symbol Makech-rescue:LM1117-SOT--Ogaki-rescue-Makech-rescue-Makech-rescue-Makech-rescue-Makech-rescue -> Makech-rescue:LM1117-SOT--Ogaki-rescue-Makech-rescue-Makech-rescue-Makech-rescue-Makech-rescue-Makech-rescue
- X1: symbol Makech-rescue:Screw_Terminal_1x02--Ogaki-rescue-Makech-rescue-Makech-rescue-Makech-rescue-Makech-rescue -> Makech-rescue:Screw_Terminal_1x02--Ogaki-rescue-Makech-rescue-Makech-rescue-Makech-rescue-Makech-rescue-Makech-rescue
- XH3, XH4: symbol Makech-rescue:CONN_01X05--Ogaki-rescue-Makech-rescue-Makech-rescue-Makech-rescue-Makech-rescue -> Makech-rescue:CONN_01X05--Ogaki-rescue-Makech-rescue-Makech-rescue-Makech-rescue-Makech-rescue-Makech-rescue
- Z1: symbol Makech-rescue:buzzer--Ogaki-rescue-Makech-rescue-Makech-rescue-Makech-rescue-Makech-rescue -> Makech-rescue:buzzer--Ogaki-rescue-Makech-rescue-Makech-rescue-Makech-rescue-Makech-rescue-Makech-rescue
Connections:
- wire segments 380 -> 384
- no-connect marks 1 -> 9

Commit message: Eliminate unnecessary elements
Parts:
- removed D1.1: ZENER, Diodes_SMD:D_0603, symbol Makech-rescue:ZENER--Ogaki-rescue-Makech-rescue-Makech-rescue-Makech-rescue-Mak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
- removed F1.1: FUSE, Resistors_SMD:R_1206_HandSoldering, symbol Makech-rescue:FUSE--Ogaki-rescue-Makech-rescue-Makech-rescue-Makech-rescue-Make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
- J3: footprint (none) -> Pines:610X1221821
- R6, R7: footprint (none) -> Resistors_SMD:R_0805_HandSoldering
- U2: renamed from U?; footprint QFP50P900X900X120-48N -> Housings_QFP:TQFP-48_7x7mm_Pitch0.5mm
Connections:
- wire segments 384 -> 376
Other:
- note added: "NOTA: Revisar \ndiodo \nde proteccion"
- note removed: "Choose on X.1 --> SMD, X --> THT"
- note removed: "Choose one\nCx.1 --> SMD\nCx --> THT"
- note removed: "Choose one\nRx.1 --> SMD\nRx --> THT"
- note removed: "Choose one\nSx.1 --> B3F-4050\nSx --> B3F-1050"
- note removed: "NOTA: Revisar \ndiodos \nde proteccion"
Changed lines of the file:
@@
 	0    -1   -1   0
 $EndComp
-Text Notes 4410 1775 0    59   ~ 0
-Choose one\nRx.1 --> SMD\nRx  -->  THT
 $Comp
 L Makech-rescue:switch--Ogaki-rescue-Makech-rescue-Makech-rescue-Makech-rescue-Makech-rescue-Makech-rescue S5.1
@@
 Text Label 8790 1295 1    60   ~ 0
 S1
-Text Notes 8440 1040 0    59   ~ 0
-Choose one\nSx.1 --> B3F-4050\nSx  -->  B3F-1050
 $Comp
 L Makech-rescue:switch--Ogaki-rescue-Makech-rescue-Makech-rescue-Makech-rescue-Makech-rescue-Makech-rescue S3
@@
 Text Label 7570 1270 1    60   ~ 0
 S4
-Text Notes 7920 2760 0    59   ~ 0
-Choose one\nRx.1 --> SMD\nRx  -->  THT
 $Comp
 L Makech-rescue:JUMPER--Ogaki-rescue-Makech-rescue-Makech-rescue-Makech-rescue-Makech-rescue-Makech-rescue SJ2
@@
 	1    0    0    -1
 $EndComp
-Text Notes 9745 6485 0    59   ~ 0
-Choose one\nCx.1 --> SMD\nCx   --> THT
 Text Label 9330 4855 0    60   ~ 0
 D13
@@
 $EndComp
 $Comp
-L Makech-rescue:FUSE--Ogaki-rescue-Makech-rescue-Makech-rescue-Makech-rescue-Makech-rescue-Makech-rescue F1.1
-U 1 1 58BB50CA
-P 2480 6885
-F 0 "F1.1" H 2525 6970 40  0000 C CNN
-F 1 "FUSE" H 2380 6835 40  0000 C CNN
-F 2 "Resistors_SMD:R_1206_HandSoldering" H 2480 6885 60  0001 C CNN
-F 3 "" H 2480 6885 60  0000 C CNN
-	1    2480 6885
-	1    0    0    -1
-$EndComp
-$Comp
 L Makech-rescue:FUSE--Ogaki-rescue-Makech-rescue-Makech-rescue-Makech-rescue-Makech-rescue-Makech-rescue F1
 U 1 1 58BB5A4E
-P 2485 7125
-F 0 "F1" H 2535 7165 40  0000 C CNN
-F 1 "FUSE" H 2385 7075 40  0000 C CNN
-F 2 "Fuse_Holders_and_Fuses:Fuse_TE5_Littlefuse-395Series" H 2485 7125 60  0001 C CNN
-F 3 "" H 2485 7125 60  0000 C CNN
-	1    2485 7125
+P 2705 7015
+F 0 "F1" H 2755 7055 40  0000 C CNN
+F 1 "FUSE" H 2605 6965 40  0000 C CNN
+F 2 "Fuse_Holders_and_Fuses:Fuse_TE5_Littlefuse-395Series" H 2705 7015 60  0001 C CNN
+F 3 "" H 2705 7015 60  0000 C CNN
+	1    2705 7015
 	1    0    0    -1
 $EndComp
 $Comp
-L Makech-rescue:ZENER--Ogaki-rescue-Makech-rescue-Makech-rescue-Makech-rescue-Makech-rescue-Makech-rescue D1.1
-U 1 1 58BB6B77
-P 2985 7285
-F 0 "D1.1" H 2985 7355 40  0000 C CNN
-F 1 "ZENER" H 2985 7185 40  0001 C CNN
-F 2 "Diodes_SMD:D_0603" H 2985 7285 60  0001 C CNN
-F 3 "" H 2985 7285 60  0000 C CNN
-F 4 "S-152T" H 2985 7285 50  0001 C CNN "manf#"
-	1    2985 7285
-	0    -1   -1   0
-$EndComp
-$Comp
 L Makech-rescue:ZENER--Ogaki-rescue-Makech-rescue-Makech-rescue-Makech-rescue-Makech-rescue-Makech-rescue D1
 U 1 1 58BB6DB1
@@
 	1    0    0    -1
 $EndComp
-Text Notes 3025 7635 2    60   ~ 0
-Choose on X.1 --> SMD,  X --> THT
 $Comp
 L Makech-rescue:CONN_01X05--Ogaki-rescue-Makech-rescue-Makech-rescue-Makech-rescue-Makech-rescue-Makech-rescue XH4
@@
 	1015 6885 2105 6885
 Wire Wire Line
-	2105 6885 2105 7125
-Wire Wire Line
 	2020 7125 2105 7125
 Wire Wire Line
@@
 Wire Wire Line
 	2105 7225 2020 7225
-Connection ~ 2105 6885
-Connection ~ 2105 7125
-Wire Wire Line
-	2735 7125 2635 7125
-Wire Wire Line
-	2735 6885 2735 7015
-Wire Wire Line
-	2735 6885 2630 6885
 Connection ~ 2105 7455
-Connection ~ 2985 7455
 Wire Wire Line
 	3035 7510 3035 7455
 Connection ~ 3035 7455
 Wire Wire Line
-	2735 7015 2985 7015
-Wire Wire Line
-	2985 7015 2985 7185
-Connection ~ 2735 7015
-Wire Wire Line
 	3080 7015 3080 7185
-Connection ~ 2985 7015
 Wire Wire Line
 	3080 7455 3080 7335
-Wire Wire Line
-	2985 7335 2985 7455
 Connection ~ 3080 7015
 Wire Wire Line
@@
 	8600 5940 8600 6295
 Wire Wire Line
-	2105 6885 2330 6885
-Wire Wire Line
-	2105 7125 2335 7125
-Wire Wire Line
-	2105 7455 2985 7455
-Wire Wire Line
-	2985 7455 3035 7455
-Wire Wire Line
 	3035 7455 3080 7455
 Wire Wire Line
-	2735 7015 2735 7125
-Wire Wire Line
-	2985 7015 3080 7015
-Wire Wire Line
 	3080 7015 3315 7015
 Wire Wire Line
@@
 $EndComp
 Text Notes 3350 7615 0    60   ~ 0
-NOTA: Revisar \ndiodos \nde proteccion
+NOTA: Revisar \ndiodo \nde proteccion
 $Comp
 L Makech-rescue:SW_Push-Switch-Makech-rescue-Makech-rescue-Makech-rescue-Makech-rescue SW1
@@
 F 0 "J3" H 7130 5867 50  0000 C CNN
 F 1 "ESP32-Exp" H 7130 5776 50  0000 C CNN
-F 2 "" H 7080 5450 50  0001 C CNN
+F 2 "Pines:610X1221821" H 7080 5450 50  0001 C CNN
 F 3 "~" H 7080 5450 50  0001 C CNN
 	1    7080 5450
@@
 F 0 "R6" H 6689 5026 50  0000 L CNN
 F 1 "10K" H 6689 4935 50  0000 L CNN
-F 2 "" H 6630 4980 50  0001 C CNN
+F 2 "Resistors_SMD:R_0805_HandSoldering" H 6630 4980 50  0001 C CNN
 F 3 "~" H 6630 4980 50  0001 C CNN
 	1    6630 4980
@@
 F 0 "R7" H 8224 5926 50  0000 L CNN
 F 1 "10K" H 8224 5835 50  0000 L CNN
-F 2 "" H 8165 5880 50  0001 C CNN
+F 2 "Resistors_SMD:R_0805_HandSoldering" H 8165 5880 50  0001 C CNN
 F 3 "~" H 8165 5880 50  0001 C CNN
 	1    8165 5880
@@
 ESP_CS
 $Comp
-L electroniccats:ATSAMD21G18A-AU U?
+L electroniccats:ATSAMD21G18A-AU U2
 U 1 1 5CBBAA5C
 P 2120 2905
-F 0 "U?" H 2120 4772 50  0000 C CNN
+F 0 "U2" H 2120 4772 50  0000 C CNN
 F 1 "ATSAMD21G18A-AU" H 2120 4681 50  0000 C CNN
-F 2 "QFP50P900X900X120-48N" H 2120 2905 50  0001 L BNN
+F 2 "Housings_QFP:TQFP-48_7x7mm_Pitch0.5mm" H 2120 2905 50  0001 L BNN
 F 3 "3.01 USD" H 2120 2905 50  0001 L BNN
 F 4 "Microchip" H 2120 2905 50  0001 L BNN "Campo4"
@@
 NoConn ~ 2820 2805
 NoConn ~ 2820 2905
+Wire Wire Line
+	2555 7015 2105 7015
+Wire Wire Line
+	2105 6885 2105 7015
+Connection ~ 2105 7015
+Wire Wire Line
+	2105 7015 2105 7125
+Wire Wire Line
+	2105 7455 3035 7455
+Wire Wire Line
+	2855 7015 3080 7015
 $EndSCHEMATC

Commit message: BOM
Parts:
- removed JP2: CONN_01X02, Pines:61300211121, symbol Makech-rescue:CONN_01X02--Ogaki-rescue-Makech-rescue-Makech-rescue-Makech-rescu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
- removed S1.1, S2.1, S3.1, S4.1, S5.1: switch, Switch:SW_PUSH_6mm, symbol Makech-rescue:switch--Ogaki-rescue-Makech-rescue-Makech-rescue-Makech-rescue-Ma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
- C1, C5, C6: symbol Makech-rescue:C_Small-Device-Makech-rescue-Makech-rescue-Makech-rescue-Makech-rescue -> Makech-rescue:C_Small-Device-Makech-rescue-Makech-rescue-Makech-rescue-Makech-rescue-Makech-rescue
- C2, C2.1, C3, C3.1, C4, C4.1: symbol Makech-rescue:C-RESCUE-Ogaki--Ogaki-rescue-Makech-rescue-Makech-rescue-Makech-rescue-Makech-rescue-Makech-rescue -> Makech-rescue:C-RESCUE-Ogaki--Ogaki-rescue-Makech-rescue-Makech-rescue-Makech-rescue-Makech-rescue-Makech-rescue-Makech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
- D1: footprint Diodes_ThroughHole:D_DO-41_SOD81_P10.16mm_Horizontal -> Diode_SMD:D_0805_2012Metric_Castellated; symbol Makech-rescue:ZENER--Ogaki-rescue-Makech-rescue-Makech-rescue-Makech-rescue-Makech-rescue-Makech-rescue -> Makech-rescue:ZENER--Ogaki-rescue-Makech-rescue-Makech-rescue-Makech-rescue-Makech-rescue-Makech-rescue-Makech-rescue; manf# (none) -> BZY55C4V7 RYG
- D2, D3: symbol Makech-rescue:D_Schottky-Device-Makech-rescue-Makech-rescue-Makech-rescue-Makech-rescue -> Makech-rescue:D_Schottky-Device-Makech-rescue-Makech-rescue-Makech-rescue-Makech-rescue-Makech-rescue; manf# (none) -> STPS1L60ZFY
- F1: symbol Makech-rescue:FUSE--Ogaki-rescue-Makech-rescue-Makech-rescue-Makech-rescue-Makech-rescue-Makech-rescue -> Makech-rescue:FUSE--Ogaki-rescue-Makech-rescue-Makech-rescue-Makech-rescue-Makech-rescue-Makech-rescue-Makech-rescue; manf# (none) -> 0ZCF0050FF2C
- F2: symbol Makech-rescue:Fuse-Device-Makech-rescue-Makech-rescue-Makech-rescue-Makech-rescue -> Makech-rescue:Fuse-Device-Makech-rescue-Makech-rescue-Makech-rescue-Makech-rescue-Makech-rescue; manf# (none) -> 0ZCG0030FF2C
- IC1: symbol Makech-rescue:ULN2803--Ogaki-rescue-Makech-rescue-Makech-rescue-Makech-rescue-Makech-rescue-Makech-rescue -> Makech-rescue:ULN2803--Ogaki-rescue-Makech-rescue-Makech-rescue-Makech-rescue-Makech-rescue-Makech-rescue-Makech-rescue
- J1: symbol Makech-rescue:USB_B_Micro-Connector-Makech-rescue-Makech-rescue-Makech-rescue-Makech-rescue -> Makech-rescue:USB_B_Micro-Connector-Makech-rescue-Makech-rescue-Makech-rescue-Makech-rescue-Makech-rescue; manf# KMMX-BSMT35S-B30TR -> 629105150521
- J2: symbol Makech-rescue:Conn_02x02_Counter_Clockwise-Connector_Generic-Makech-rescue-Makech-rescue-Makech-rescue-Makech-rescue -> Makech-rescue:Conn_02x02_Counter_Clockwise-Connector_Generic-Makech-rescue-Makech-rescue-Makech-rescue-Makech-rescue-Ma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
- J3: manf# (none) -> ESP32
- JP1: symbol Makech-rescue:CONN_01X02--Ogaki-rescue-Makech-rescue-Makech-rescue-Makech-rescue-Makech-rescue-Makech-rescue -> Makech-rescue:CONN_01X02--Ogaki-rescue-Makech-rescue-Makech-rescue-Makech-rescue-Makech-rescue-Makech-rescue-Makech-res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
- LED1, LED1.1, LED2, LED2.1, LED3, LED3.1, LED4, LED4.1: symbol Makech-rescue:LED-RESCUE-Ogaki--Ogaki-rescue-Makech-rescue-Makech-rescue-Makech-rescue-Makech-rescue-Makech-rescue -> Makech-rescue:LED-RESCUE-Ogaki--Ogaki-rescue-Makech-rescue-Makech-rescue-Makech-rescue-Makech-rescue-Makech-rescue-Make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
- R1, R2, R3, R4, R5: symbol Makech-rescue:R-SIL_8NB--Ogaki-rescue-Makech-rescue-Makech-rescue-Makech-rescue-Makech-rescue-Makech-rescue -> Makech-rescue:R-SIL_8NB--Ogaki-rescue-Makech-rescue-Makech-rescue-Makech-rescue-Makech-rescue-Makech-rescue-Makech-resc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
- R1.1, R10.1, R2.2, R3.1, R4.1, R5.1, R6.1, R7.1, R8.1, R9.1: symbol Makech-rescue:R-RESCUE-Ogaki--Ogaki-rescue-Makech-rescue-Makech-rescue-Makech-rescue-Makech-rescue-Makech-rescue -> Makech-rescue:R-RESCUE-Ogaki--Ogaki-rescue-Makech-rescue-Makech-rescue-Makech-rescue-Makech-rescue-Makech-rescue-Makech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
- R6, R7: manf# (none) -> CRCW080510K0FKEAC
- S1, S2, S4, S5: footprint Switch:Button -> Button_Switch_THT:SW_PUSH-12mm_Wuerth-430476085716; symbol Makech-rescue:switch--Ogaki-rescue-Makech-rescue-Makech-rescue-Makech-rescue-Makech-rescue-Makech-rescue -> Makech-rescue:switch--Ogaki-rescue-Makech-rescue-Makech-rescue-Makech-rescue-Makech-rescue-Makech-rescue-Makech-rescue; manf# KSC441G70SHLFSPF -> 50pcs Tactile Push Button Switch Momentary Tact & Cap Assor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
- S3: footprint Switch:Button -> Button_Switch_THT:SW_PUSH-12mm; symbol Makech-rescue:switch--Ogaki-rescue-Makech-rescue-Makech-rescue-Makech-rescue-Makech-rescue-Makech-rescue -> Makech-rescue:switch--Ogaki-rescue-Makech-rescue-Makech-rescue-Makech-rescue-Makech-rescue-Makech-rescue-Makech-rescue; manf# KSC441G70SHLFSPF -> 50pcs Tactile Push Button Switch Momentary Tact & Cap Assor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
- S7: symbol Makech-rescue:switch--Ogaki-rescue-Makech-rescue-Makech-rescue-Makech-rescue-Makech-rescue-Makech-rescue -> Makech-rescue:switch--Ogaki-rescue-Makech-rescue-Makech-rescue-Makech-rescue-Makech-rescue-Makech-rescue-Makech-rescue
- SJ2: symbol Makech-rescue:JUMPER--Ogaki-rescue-Makech-rescue-Makech-rescue-Makech-rescue-Makech-rescue-Makech-rescue -> Makech-rescue:JUMPER--Ogaki-rescue-Makech-rescue-Makech-rescue-Makech-rescue-Makech-rescue-Makech-rescue-Makech-rescue
- SW1: footprint TIH:SW_B3U-1000P -> Button_Switch_SMD:SW_SPST_TL3342; symbol Makech-rescue:SW_Push-Switch-Makech-rescue-Makech-rescue-Makech-rescue-Makech-rescue -> Makech-rescue:SW_Push-Switch-Makech-rescue-Makech-rescue-Makech-rescue-Makech-rescue-Makech-rescue; manf# (none) -> Boton Generico
- U1: symbol Makech-rescue:CONN_01X04--Ogaki-rescue-Makech-rescue-Makech-rescue-Makech-rescue-Makech-rescue-Makech-rescue -> Makech-rescue:CONN_01X04--Ogaki-rescue-Makech-rescue-Makech-rescue-Makech-rescue-Makech-rescue-Makech-rescue-Makech-res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
- U2: symbol electroniccats:ATSAMD21G18A-AU -> Makech-rescue:ATSAMD21G18A-AU-electroniccats
- U6: symbol Makech-rescue:LM1117-SOT--Ogaki-rescue-Makech-rescue-Makech-rescue-Makech-rescue-Makech-rescue-Makech-rescue -> Makech-rescue:LM1117-SOT--Ogaki-rescue-Makech-rescue-Makech-rescue-Makech-rescue-Makech-rescue-Makech-rescue-Makech-res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
- X1: symbol Makech-rescue:Screw_Terminal_1x02--Ogaki-rescue-Makech-rescue-Makech-rescue-Makech-rescue-Makech-rescue-Makech-rescue -> Makech-rescue:Screw_Terminal_1x02--Ogaki-rescue-Makech-rescue-Makech-rescue-Makech-rescue-Makech-rescue-Makech-rescue-M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
- XH3, XH4: symbol Makech-rescue:CONN_01X05--Ogaki-rescue-Makech-rescue-Makech-rescue-Makech-rescue-Makech-rescue-Makech-rescue -> Makech-rescue:CONN_01X05--Ogaki-rescue-Makech-rescue-Makech-rescue-Makech-rescue-Makech-rescue-Makech-rescue-Makech-res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; manf# (none) -> B5B-XH-A (LF)(SN)
- Z1: symbol Makech-rescue:buzzer--Ogaki-rescue-Makech-rescue-Makech-rescue-Makech-rescue-Makech-rescue-Makech-rescue -> Makech-rescue:buzzer--Ogaki-rescue-Makech-rescue-Makech-rescue-Makech-rescue-Makech-rescue-Makech-rescue-Makech-rescue; manf# (none) -> F/CM12P-LF
Connections:
- wire segments 376 -> 331

Commit message: BOM
Parts:
- F1: footprint Fuse_Holders_and_Fuses:Fuse_TE5_Littlefuse-395Series -> Fuse:Fuse_0805_2012Metric
- F2: footprint (none) -> Fuse:Fuse_0805_2012Metric
- JP1: manf# (none) -> 61300211121
- XH3, XH4: footprint user_molex:B5B-XH-A -> Connector_Molex:Molex_SPOX_5267-05A_1x05_P2.50mm_Vertical
Changed lines of the file:
@@
 F 2 "Pines:61300211121" H 4300 5565 50  0001 C CNN
 F 3 "" H 4300 5565 50  0000 C CNN
+F 4 "61300211121" H 4300 5565 50  0001 C CNN "manf#"
 	1    4300 5565
 	1    0    0    -1
@@
 F 0 "F1" H 2755 7055 40  0000 C CNN
 F 1 "FUSE" H 2605 6965 40  0000 C CNN
-F 2 "Fuse_Holders_and_Fuses:Fuse_TE5_Littlefuse-395Series" H 2705 7015 60  0001 C CNN
+F 2 "Fuse:Fuse_0805_2012Metric" H 2705 7015 60  0001 C CNN
 F 3 "" H 2705 7015 60  0000 C CNN
 F 4 "0ZCF0050FF2C" H 2705 7015 50  0001 C CNN "manf#"
@@
 F 0 "XH4" H 11045 6005 50  0000 C CNN
 F 1 "CONN_01X05" V 11145 5705 50  0001 C CNN
-F 2 "user_molex:B5B-XH-A" H 11045 5705 50  0001 C CNN
+F 2 "Connector_Molex:Molex_SPOX_5267-05A_1x05_P2.50mm_Vertical" H 11045 5705 50  0001 C CNN
 F 3 "" H 11045 5705 50  0000 C CNN
 F 4 "B5B-XH-A (LF)(SN) " H 11045 5705 50  0001 C CNN "manf#"
@@
 F 0 "XH3" H 11045 4520 50  0000 C CNN
 F 1 "CONN_01X05" V 11145 4810 50  0001 C CNN
-F 2 "user_molex:B5B-XH-A" H 11045 4810 50  0001 C CNN
+F 2 "Connector_Molex:Molex_SPOX_5267-05A_1x05_P2.50mm_Vertical" H 11045 4810 50  0001 C CNN
 F 3 "" H 11045 4810 50  0000 C CNN
 F 4 "B5B-XH-A (LF)(SN) " H 11045 4810 50  0001 C CNN "manf#"
@@
 F 0 "F2" V 3103 5590 50  0000 C CNN
 F 1 "0.5" V 3194 5590 50  0000 C CNN
-F 2 "" V 3230 5590 50  0001 C CNN
+F 2 "Fuse:Fuse_0805_2012Metric" V 3230 5590 50  0001 C CNN
 F 3 "~" H 3300 5590 50  0001 C CNN
 F 4 "0ZCG0030FF2C" V 3300 5590 50  0001 C CNN "manf#"
