File: Makech/hardware/KiCad files/Makech.sch (KiCad schematic (older format))
At the start: 59 parts, among them IC1 ULN2803, J1 USB_B_Micro, J2 SWD programmer, J3 ESP32-Exp, SW1 RST, U1 CONN_01X04, U2 ATSAMD21G18A-AU, U6 AP2114_3.3v, X1 Screw_Terminal_1x02

Commit message: Fix error library index
Parts:
- C1, C5, C6: symbol Makech-rescue:C_Small-Device-Makech-rescue-Makech-rescue-Makech-rescue-Makech-rescue-Makech-rescue -> Makech-rescue:C_Small-Device-Makech-rescue-Makech-rescue-Makech-rescue-Makech-rescue-Makech-rescue-Makech-rescue
- C2, C2.1, C3, C3.1, C4, C4.1: symbol Makech-rescue:C-RESCUE-Ogaki--Ogaki-rescue-Makech-rescue-Makech-rescue-Makech-rescue-Makech-rescue-Makech-rescue-Makech-rescue -> Makech-rescue:C-RESCUE-Ogaki--Ogaki-rescue-Makech-rescue-Makech-rescue-Makech-rescue-Makech-rescue-Makech-rescue-Makech-rescue-Makech-rescue
- D1: symbol Makech-rescue:ZENER--Ogaki-rescue-Makech-rescue-Makech-rescue-Makech-rescue-Makech-rescue-Makech-rescue-Makech-rescue -> Makech-rescue:ZENER--Ogaki-rescue-Makech-rescue-Makech-rescue-Makech-rescue-Makech-rescue-Makech-rescue-Makech-rescue-M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
- D2, D3: symbol Makech-rescue:D_Schottky-Device-Makech-rescue-Makech-rescue-Makech-rescue-Makech-rescue-Makech-rescue -> Makech-rescue:D_Schottky-Device-Makech-rescue-Makech-rescue-Makech-rescue-Makech-rescue-Makech-rescue-Makech-rescue
- F1: symbol Makech-rescue:FUSE--Ogaki-rescue-Makech-rescue-Makech-rescue-Makech-rescue-Makech-rescue-Makech-rescue-Makech-rescue -> Makech-rescue:FUSE--Ogaki-rescue-Makech-rescue-Makech-rescue-Makech-rescue-Makech-rescue-Makech-rescue-Makech-rescue-Ma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
- F2: symbol Makech-rescue:Fuse-Device-Makech-rescue-Makech-rescue-Makech-rescue-Makech-rescue-Makech-rescue -> Makech-rescue:Fuse-Device-Makech-rescue-Makech-rescue-Makech-rescue-Makech-rescue-Makech-rescue-Makech-rescue
- IC1: symbol Makech-rescue:ULN2803--Ogaki-rescue-Makech-rescue-Makech-rescue-Makech-rescue-Makech-rescue-Makech-rescue-Makech-rescue -> Makech-rescue:ULN2803--Ogaki-rescue-Makech-rescue-Makech-rescue-Makech-rescue-Makech-rescue-Makech-rescue-Makech-rescue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
- J1: symbol Makech-rescue:USB_B_Micro-Connector-Makech-rescue-Makech-rescue-Makech-rescue-Makech-rescue-Makech-rescue -> Makech-rescue:USB_B_Micro-Connector-Makech-rescue-Makech-rescue-Makech-rescue-Makech-rescue-Makech-rescue-Makech-rescue
- J2: symbol Makech-rescue:Conn_02x02_Counter_Clockwise-Connector_Generic-Makech-rescue-Makech-rescue-Makech-rescue-Makech-rescue-Makech-rescue -> Makech-rescue:Conn_02x02_Counter_Clockwise-Connector_Generic-Makech-rescue-Makech-rescue-Makech-rescue-Makech-rescue-Makech-rescue-Makech-rescue
- JP1: symbol Makech-rescue:CONN_01X02--Ogaki-rescue-Makech-rescue-Makech-rescue-Makech-rescue-Makech-rescue-Makech-rescue-Makech-rescue -> Makech-rescue:CONN_01X02--Ogaki-rescue-Makech-rescue-Makech-rescue-Makech-rescue-Makech-rescue-Makech-rescue-Makech-rescue-Makech-rescue
- LED1, LED1.1, LED2, LED2.1, LED3, LED3.1, LED4, LED4.1: symbol Makech-rescue:LED-RESCUE-Ogaki--Ogaki-rescue-Makech-rescue-Makech-rescue-Makech-rescue-Makech-rescue-Makech-rescue-Makech-rescue -> Makech-rescue:LED-RESCUE-Ogaki--Ogaki-rescue-Makech-rescue-Makech-rescue-Makech-rescue-Makech-rescue-Makech-rescue-Makech-rescue-Makech-rescue
- R1, R2, R3, R4, R5: symbol Makech-rescue:R-SIL_8NB--Ogaki-rescue-Makech-rescue-Makech-rescue-Makech-rescue-Makech-rescue-Makech-rescue-Makech-rescue -> Makech-rescue:R-SIL_8NB--Ogaki-rescue-Makech-rescue-Makech-rescue-Makech-rescue-Makech-rescue-Makech-rescue-Makech-rescue-Makech-rescue
- R1.1, R10.1, R2.2, R3.1, R4.1, R5.1, R6.1, R7.1, R8.1, R9.1: symbol Makech-rescue:R-RESCUE-Ogaki--Ogaki-rescue-Makech-rescue-Makech-rescue-Makech-rescue-Makech-rescue-Makech-rescue-Makech-rescue -> Makech-rescue:R-RESCUE-Ogaki--Ogaki-rescue-Makech-rescue-Makech-rescue-Makech-rescue-Makech-rescue-Makech-rescue-Makech-rescue-Makech-rescue
- S1, S2, S3, S4, S5, S7: symbol Makech-rescue:switch--Ogaki-rescue-Makech-rescue-Makech-rescue-Makech-rescue-Makech-rescue-Makech-rescue-Makech-rescue -> Makech-rescue:switch--Ogaki-rescue-Makech-rescue-Makech-rescue-Makech-rescue-Makech-rescue-Makech-rescue-Makech-rescue-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
- SJ2: symbol Makech-rescue:JUMPER--Ogaki-rescue-Makech-rescue-Makech-rescue-Makech-rescue-Makech-rescue-Makech-rescue-Makech-rescue -> Makech-rescue:JUMPER--Ogaki-rescue-Makech-rescue-Makech-rescue-Makech-rescue-Makech-rescue-Makech-rescue-Makech-rescue-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
- SW1: symbol Makech-rescue:SW_Push-Switch-Makech-rescue-Makech-rescue-Makech-rescue-Makech-rescue-Makech-rescue -> Makech-rescue:SW_Push-Switch-Makech-rescue-Makech-rescue-Makech-rescue-Makech-rescue-Makech-rescue-Makech-rescue
- U1: symbol Makech-rescue:CONN_01X04--Ogaki-rescue-Makech-rescue-Makech-rescue-Makech-rescue-Makech-rescue-Makech-rescue-Makech-rescue -> Makech-rescue:CONN_01X04--Ogaki-rescue-Makech-rescue-Makech-rescue-Makech-rescue-Makech-rescue-Makech-rescue-Makech-rescue-Makech-rescue
- U2: symbol Makech-rescue:ATSAMD21G18A-AU-electroniccats -> Makech-rescue:ATSAMD21G18A-AU-electroniccats-Makech-rescue
- U6: symbol Makech-rescue:LM1117-SOT--Ogaki-rescue-Makech-rescue-Makech-rescue-Makech-rescue-Makech-rescue-Makech-rescue-Makech-rescue -> Makech-rescue:LM1117-SOT--Ogaki-rescue-Makech-rescue-Makech-rescue-Makech-rescue-Makech-rescue-Makech-rescue-Makech-rescue-Makech-rescue
- X1: symbol Makech-rescue:Screw_Terminal_1x02--Ogaki-rescue-Makech-rescue-Makech-rescue-Makech-rescue-Makech-rescue-Makech-rescue-Makech-rescue -> Makech-rescue:Screw_Terminal_1x02--Ogaki-rescue-Makech-rescue-Makech-rescue-Makech-rescue-Makech-rescue-Makech-rescue-Makech-rescue-Makech-rescue
- XH3, XH4: symbol Makech-rescue:CONN_01X05--Ogaki-rescue-Makech-rescue-Makech-rescue-Makech-rescue-Makech-rescue-Makech-rescue-Makech-rescue -> Makech-rescue:CONN_01X05--Ogaki-rescue-Makech-rescue-Makech-rescue-Makech-rescue-Makech-rescue-Makech-rescue-Makech-rescue-Makech-rescue
- Z1: symbol Makech-rescue:buzzer--Ogaki-rescue-Makech-rescue-Makech-rescue-Makech-rescue-Makech-rescue-Makech-rescue-Makech-rescue -> Makech-rescue:buzzer--Ogaki-rescue-Makech-rescue-Makech-rescue-Makech-rescue-Makech-rescue-Makech-rescue-Makech-rescue-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
Connections:
- wire segments 331 -> 330

Commit message: remove components x.1
Parts:
- removed LED1.1, LED2.1, LED3.1, LED4.1: L, LED_SMD:LED_0805_2012Metric, symbol Makech-rescue:LED-RESCUE-Ogaki--Ogaki-rescue-Makech-rescue-Makech-rescue-Makech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
- removed R1.1, R2.2, R3.1, R4.1, R5.1, R7.1: 10K, Resistors_SMD:R_0805_HandSoldering, symbol Makech-rescue:R-RESCUE-Ogaki--Ogaki-rescue-Makech-rescue-Makech-rescue-Makech-r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
- removed R10.1: 100R, Resistors_SMD:R_0805_HandSoldering, symbol Makech-rescue:R-RESCUE-Ogaki--Ogaki-rescue-Makech-rescue-Makech-rescue-Makech-r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
- removed R6.1, R8.1, R9.1: 1K, Resistors_SMD:R_0805_HandSoldering, symbol Makech-rescue:R-RESCUE-Ogaki--Ogaki-rescue-Makech-rescue-Makech-rescue-Makech-r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
Connections:
- wire segments 330 -> 280

Commit message: cache lib
Parts:
- C1, C5, C6: symbol Makech-rescue:C_Small-Device-Makech-rescue-Makech-rescue-Makech-rescue-Makech-rescue-Makech-rescue-Makech-rescue -> Makech-rescue:C_Small-Device-Makech-rescue-Makech-rescue-Makech-rescue-Makech-rescue-Makech-rescue-Makech-rescue-Makech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
- C2, C2.1, C3, C3.1, C4, C4.1: symbol Makech-rescue:C-RESCUE-Ogaki--Ogaki-rescue-Makech-rescue-Makech-rescue-Makech-rescue-Makech-rescue-Makech-rescue-Makech-rescue-Makech-rescue -> Makech-rescue:C-RESCUE-Ogaki--Ogaki-rescue-Makech-rescue-Makech-rescue-Makech-rescue-Makech-rescue-Makech-rescue-Makech-rescue-Makech-rescue-Makech-rescue
- D1: symbol Makech-rescue:ZENER--Ogaki-rescue-Makech-rescue-Makech-rescue-Makech-rescue-Makech-rescue-Makech-rescue-Makech-rescue-Makech-rescue -> Makech-rescue:ZENER--Ogaki-rescue-Makech-rescue-Makech-rescue-Makech-rescue-Makech-rescue-Makech-rescue-Makech-rescue-Makech-rescue-Makech-rescue
- D2, D3: symbol Makech-rescue:D_Schottky-Device-Makech-rescue-Makech-rescue-Makech-rescue-Makech-rescue-Makech-rescue-Makech-rescue -> Makech-rescue:D_Schottky-Device-Makech-rescue-Makech-rescue-Makech-rescue-Makech-rescue-Makech-rescue-Makech-rescue-Mak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
- F1: symbol Makech-rescue:FUSE--Ogaki-rescue-Makech-rescue-Makech-rescue-Makech-rescue-Makech-rescue-Makech-rescue-Makech-rescue-Makech-rescue -> Makech-rescue:FUSE--Ogaki-rescue-Makech-rescue-Makech-rescue-Makech-rescue-Makech-rescue-Makech-rescue-Makech-rescue-Makech-rescue-Makech-rescue
- F2: symbol Makech-rescue:Fuse-Device-Makech-rescue-Makech-rescue-Makech-rescue-Makech-rescue-Makech-rescue-Makech-rescue -> Makech-rescue:Fuse-Device-Makech-rescue-Makech-rescue-Makech-rescue-Makech-rescue-Makech-rescue-Makech-rescue-Makech-re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
- IC1: symbol Makech-rescue:ULN2803--Ogaki-rescue-Makech-rescue-Makech-rescue-Makech-rescue-Makech-rescue-Makech-rescue-Makech-rescue-Makech-rescue -> Makech-rescue:ULN2803--Ogaki-rescue-Makech-rescue-Makech-rescue-Makech-rescue-Makech-rescue-Makech-rescue-Makech-rescue-Makech-rescue-Makech-rescue
- J1: symbol Makech-rescue:USB_B_Micro-Connector-Makech-rescue-Makech-rescue-Makech-rescue-Makech-rescue-Makech-rescue-Makech-rescue -> Makech-rescue:USB_B_Micro-Connector-Makech-rescue-Makech-rescue-Makech-rescue-Makech-rescue-Makech-rescue-Makech-rescue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
- J2: symbol Makech-rescue:Conn_02x02_Counter_Clockwise-Connector_Generic-Makech-rescue-Makech-rescue-Makech-rescue-Makech-rescue-Makech-rescue-Makech-rescue -> Makech-rescue:Conn_02x02_Counter_Clockwise-Connector_Generic-Makech-rescue-Makech-rescue-Makech-rescue-Makech-rescue-Makech-rescue-Makech-rescue-Makech-rescue
- JP1: symbol Makech-rescue:CONN_01X02--Ogaki-rescue-Makech-rescue-Makech-rescue-Makech-rescue-Makech-rescue-Makech-rescue-Makech-rescue-Makech-rescue -> Makech-rescue:CONN_01X02--Ogaki-rescue-Makech-rescue-Makech-rescue-Makech-rescue-Makech-rescue-Makech-rescue-Makech-rescue-Makech-rescue-Makech-rescue
- LED1, LED2, LED3, LED4: symbol Makech-rescue:LED-RESCUE-Ogaki--Ogaki-rescue-Makech-rescue-Makech-rescue-Makech-rescue-Makech-rescue-Makech-rescue-Makech-rescue-Makech-rescue -> Makech-rescue:LED-RESCUE-Ogaki--Ogaki-rescue-Makech-rescue-Makech-rescue-Makech-rescue-Makech-rescue-Makech-rescue-Makech-rescue-Makech-rescue-Makech-rescue
- R1, R2, R3, R4, R5: symbol Makech-rescue:R-SIL_8NB--Ogaki-rescue-Makech-rescue-Makech-rescue-Makech-rescue-Makech-rescue-Makech-rescue-Makech-rescue-Makech-rescue -> Makech-rescue:R-SIL_8NB--Ogaki-rescue-Makech-rescue-Makech-rescue-Makech-rescue-Makech-rescue-Makech-rescue-Makech-rescue-Makech-rescue-Makech-rescue
- S1, S2, S3, S4, S5, S7: symbol Makech-rescue:switch--Ogaki-rescue-Makech-rescue-Makech-rescue-Makech-rescue-Makech-rescue-Makech-rescue-Makech-rescue-Makech-rescue -> Makech-rescue:switch--Ogaki-rescue-Makech-rescue-Makech-rescue-Makech-rescue-Makech-rescue-Makech-rescue-Makech-rescue-Makech-rescue-Makech-rescue
- SJ2: symbol Makech-rescue:JUMPER--Ogaki-rescue-Makech-rescue-Makech-rescue-Makech-rescue-Makech-rescue-Makech-rescue-Makech-rescue-Makech-rescue -> Makech-rescue:JUMPER--Ogaki-rescue-Makech-rescue-Makech-rescue-Makech-rescue-Makech-rescue-Makech-rescue-Makech-rescue-Makech-rescue-Makech-rescue
- SW1: symbol Makech-rescue:SW_Push-Switch-Makech-rescue-Makech-rescue-Makech-rescue-Makech-rescue-Makech-rescue-Makech-rescue -> Makech-rescue:SW_Push-Switch-Makech-rescue-Makech-rescue-Makech-rescue-Makech-rescue-Makech-rescue-Makech-rescue-Makech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
- U1: symbol Makech-rescue:CONN_01X04--Ogaki-rescue-Makech-rescue-Makech-rescue-Makech-rescue-Makech-rescue-Makech-rescue-Makech-rescue-Makech-rescue -> Makech-rescue:CONN_01X04--Ogaki-rescue-Makech-rescue-Makech-rescue-Makech-rescue-Makech-rescue-Makech-rescue-Makech-rescue-Makech-rescue-Makech-rescue
- U2: symbol Makech-rescue:ATSAMD21G18A-AU-electroniccats-Makech-rescue -> Makech-rescue:ATSAMD21G18A-AU-electroniccats-Makech-rescue-Makech-rescue
- U6: symbol Makech-rescue:LM1117-SOT--Ogaki-rescue-Makech-rescue-Makech-rescue-Makech-rescue-Makech-rescue-Makech-rescue-Makech-rescue-Makech-rescue -> Makech-rescue:LM1117-SOT--Ogaki-rescue-Makech-rescue-Makech-rescue-Makech-rescue-Makech-rescue-Makech-rescue-Makech-rescue-Makech-rescue-Makech-rescue
- X1: symbol Makech-rescue:Screw_Terminal_1x02--Ogaki-rescue-Makech-rescue-Makech-rescue-Makech-rescue-Makech-rescue-Makech-rescue-Makech-rescue-Makech-rescue -> Makech-rescue:Screw_Terminal_1x02--Ogaki-rescue-Makech-rescue-Makech-rescue-Makech-rescue-Makech-rescue-Makech-rescue-Makech-rescue-Makech-rescue-Makech-rescue
- XH3, XH4: symbol Makech-rescue:CONN_01X05--Ogaki-rescue-Makech-rescue-Makech-rescue-Makech-rescue-Makech-rescue-Makech-rescue-Makech-rescue-Makech-rescue -> Makech-rescue:CONN_01X05--Ogaki-rescue-Makech-rescue-Makech-rescue-Makech-rescue-Makech-rescue-Makech-rescue-Makech-rescue-Makech-rescue-Makech-rescue
- Z1: symbol Makech-rescue:buzzer--Ogaki-rescue-Makech-rescue-Makech-rescue-Makech-rescue-Makech-rescue-Makech-rescue-Makech-rescue-Makech-rescue -> Makech-rescue:buzzer--Ogaki-rescue-Makech-rescue-Makech-rescue-Makech-rescue-Makech-rescue-Makech-rescue-Makech-rescue-Makech-rescue-Makech-rescue

Commit message: FOOTPRINT
Parts:
- C1, C3.1, C5, C6: footprint Capacitors_SMD:C_0805_HandSoldering -> Capacitor_SMD:C_0805_2012Metric_Pad1.15x1.40mm_HandSolder
- C2.1: footprint Capacitors_SMD:C_0603_HandSoldering -> Capacitor_SMD:C_0603_1608Metric_Pad1.05x0.95mm_HandSolder
- C4.1: footprint Capacitors_SMD:C_0603_HandSoldering -> Capacitor_SMD:C_0805_2012Metric_Pad1.15x1.40mm_HandSolder
- D2, D3: footprint Diodes_SMD:D_SOD-123 -> Diode_SMD:D_SOD-123
- IC1: footprint Housings_SOIC:SOIC-18W_7.5x11.6mm_Pitch1.27mm -> Package_SO:SOIC-18W_7.5x11.6mm_P1.27mm
- J1: footprint Connect:USB_Micro-B_10103594-0001LF -> Connector_USB:USB_Micro-B_Amphenol_10103594-0001LF_Horizontal
- J2: footprint Pines:62000421121 -> Connector_PinHeader_1.00mm:PinHeader_2x02_P1.00mm_Vertical_SMD
- J3: footprint Pines:610X1221821 -> Connector_PinHeader_1.00mm:PinHeader_2x06_P1.00mm_Vertical_SMD
- JP1: footprint Pines:61300211121 -> Connector_Wire:SolderWirePad_1x02_P3.81mm_Drill0.8mm
- R6, R7: footprint Resistors_SMD:R_0805_HandSoldering -> Resistor_SMD:R_0805_2012Metric_Pad1.15x1.40mm_HandSolder
- S7: footprint Switch:on_off_Switch -> Button_Switch_THT:SW_CuK_OS102011MA1QN1_SPDT_Angled
- U1: footprint Pin_Headers:Pin_Header_Straight_1x04_Pitch2.54mm -> Connector_PinHeader_2.54mm:PinHeader_1x04_P2.54mm_Vertical
- U2: footprint Housings_QFP:TQFP-48_7x7mm_Pitch0.5mm -> Package_QFP:TQFP-48_7x7mm_P0.5mm
- U6: footprint TO_SOT_Packages_THT:TO-220_Vertical -> Package_TO_SOT_SMD:SOT-223
- XH3: footprint Connector_Molex:Molex_SPOX_5267-05A_1x05_P2.50mm_Vertical -> Connector_Molex:Molex_KK-254_AE-6410-05A_1x05_P2.54mm_Vertical
- XH4: footprint Connector_Molex:Molex_SPOX_5267-05A_1x05_P2.50mm_Vertical -> Connector_Molex:Molex_KK-254_AE-6410-04A_1x04_P2.54mm_Vertical
- Z1: footprint Buzzers_Beepers:MagneticBuzzer_StarMicronics_HMB-06_HMB-12 -> Buzzer_Beeper:MagneticBuzzer_StarMicronics_HMB-06_HMB-12
Changed lines of the file:
@@
 F 0 "JP1" H 4300 5715 50  0000 C CNN
 F 1 "CONN_01X02" V 4400 5565 50  0001 C CNN
-F 2 "Pines:61300211121" H 4300 5565 50  0001 C CNN
+F 2 "Connector_Wire:SolderWirePad_1x02_P3.81mm_Drill0.8mm" H 4300 5565 50  0001 C CNN
 F 3 "" H 4300 5565 50  0000 C CNN
 F 4 "61300211121" H 4300 5565 50  0001 C CNN "manf#"
@@
 F 0 "Z1" H 4240 6010 50  0000 L CNN
 F 1 "buzzer" H 4240 5910 50  0000 L CNN
-F 2 "Buzzers_Beepers:MagneticBuzzer_StarMicronics_HMB-06_HMB-12" H 4165 5960 60  0001 C CNN
+F 2 "Buzzer_Beeper:MagneticBuzzer_StarMicronics_HMB-06_HMB-12" H 4165 5960 60  0001 C CNN
 F 3 "" H 4165 5960 60  0000 C CNN
 F 4 "F/CM12P-LF" H 4165 5960 50  0001 C CNN "manf#"
@@
 F 0 "U1" H 5600 5460 50  0000 C CNN
 F 1 "CONN_01X04" V 5700 5210 50  0001 C CNN
-F 2 "Pin_Headers:Pin_Header_Straight_1x04_Pitch2.54mm" H 5600 5210 50  0001 C CNN
+F 2 "Connector_PinHeader_2.54mm:PinHeader_1x04_P2.54mm_Vertical" H 5600 5210 50  0001 C CNN
 F 3 "" H 5600 5210 50  0000 C CNN
 	1    5600 5210
@@
 F 0 "IC1" H 9635 5655 60  0000 C CNN
 F 1 "ULN2803" H 10095 4750 60  0000 C CNN
-F 2 "Housings_SOIC:SOIC-18W_7.5x11.6mm_Pitch1.27mm" H 9880 5205 60  0001 C CNN
+F 2 "Package_SO:SOIC-18W_7.5x11.6mm_P1.27mm" H 9880 5205 60  0001 C CNN
 F 3 "" H 9880 5205 60  0000 C CNN
 F 4 "ULN2803ADWR" H 9880 5205 50  0001 C CNN "manf#"
@@
 F 0 "C2.1" V 8730 5505 50  0000 L CNN
 F 1 "100nF" V 8865 5645 50  0000 L CNN
-F 2 "Capacitors_SMD:C_0603_HandSoldering" H 8820 5620 60  0001 C CNN
+F 2 "Capacitor_SMD:C_0603_1608Metric_Pad1.05x0.95mm_HandSolder" H 8820 5620 60  0001 C CNN
 F 3 "" H 8820 5620 60  0000 C CNN
 F 4 "08051C104J4T4A" V 8820 5620 50  0001 C CNN "manf#"
@@
 F 0 "XH4" H 11045 6005 50  0000 C CNN
 F 1 "CONN_01X05" V 11145 5705 50  0001 C CNN
-F 2 "Connector_Molex:Molex_SPOX_5267-05A_1x05_P2.50mm_Vertical" H 11045 5705 50  0001 C CNN
+F 2 "Connector_Molex:Molex_KK-254_AE-6410-04A_1x04_P2.54mm_Vertical" H 11045 5705 50  0001 C CNN
 F 3 "" H 11045 5705 50  0000 C CNN
 F 4 "B5B-XH-A (LF)(SN) " H 11045 5705 50  0001 C CNN "manf#"
@@
 F 0 "XH3" H 11045 4520 50  0000 C CNN
 F 1 "CONN_01X05" V 11145 4810 50  0001 C CNN
-F 2 "Connector_Molex:Molex_SPOX_5267-05A_1x05_P2.50mm_Vertical" H 11045 4810 50  0001 C CNN
+F 2 "Connector_Molex:Molex_KK-254_AE-6410-05A_1x05_P2.54mm_Vertical" H 11045 4810 50  0001 C CNN
 F 3 "" H 11045 4810 50  0000 C CNN
 F 4 "B5B-XH-A (LF)(SN) " H 11045 4810 50  0001 C CNN "manf#"
@@
 F 0 "S7" H 3390 6915 60  0000 C CNN
 F 1 "switch" H 3560 6665 60  0000 C CNN
-F 2 "Switch:on_off_Switch" H 3480 6915 60  0001 C CNN
+F 2 "Button_Switch_THT:SW_CuK_OS102011MA1QN1_SPDT_Angled" H 3480 6915 60  0001 C CNN
 F 3 "" H 3480 6915 60  0001 C CNN
 F 4 "1825232-1" H 3480 6915 50  0001 C CNN "manf#"
@@
 F 0 "U6" H 6000 7015 60  0000 C CNN
 F 1 "AP2114_3.3v" H 6000 6915 60  0000 C CNN
-F 2 "TO_SOT_Packages_THT:TO-220_Vertical" H 6000 6815 60  0001 C CNN
+F 2 "Package_TO_SOT_SMD:SOT-223" H 6000 6815 60  0001 C CNN
 F 3 "" H 6000 6815 60  0000 C CNN
 F 4 "AP2114HA-3.3TRG1" H 6000 6815 50  0001 C CNN "manf#"
@@
 F 0 "C3.1" V 5690 7405 50  0000 L CNN
 F 1 "10uF" V 5810 7530 50  0000 L CNN
-F 2 "Capacitors_SMD:C_0805_HandSoldering" H 5775 7520 60  0001 C CNN
+F 2 "Capacitor_SMD:C_0805_2012Metric_Pad1.15x1.40mm_HandSolder" H 5775 7520 60  0001 C CNN
 F 3 "" H 5775 7520 60  0000 C CNN
 F 4 "C0805X106K8RACAUTO" V 5775 7520 50  0001 C CNN "manf#"
@@
 F 0 "C4.1" V 6140 7450 50  0000 L CNN
 F 1 "10uF" V 6255 7295 50  0000 L CNN
-F 2 "Capacitors_SMD:C_0603_HandSoldering" H 6225 7520 60  0001 C CNN
+F 2 "Capacitor_SMD:C_0805_2012Metric_Pad1.15x1.40mm_HandSolder" H 6225 7520 60  0001 C CNN
 F 3 "" H 6225 7520 60  0000 C CNN
 F 4 "C0805X106K8RACAUTO" V 6225 7520 50  0001 C CNN "manf#"
@@
 F 0 "C1" H 3182 1921 50  0000 L CNN
 F 1 "1uF" H 3182 1830 50  0000 L CNN
-F 2 "Capacitors_SMD:C_0805_HandSoldering" H 3090 1875 50  0001 C CNN
+F 2 "Capacitor_SMD:C_0805_2012Metric_Pad1.15x1.40mm_HandSolder" H 3090 1875 50  0001 C CNN
 F 3 "~" H 3090 1875 50  0001 C CNN
 F 4 "CGA4J1X8R1E105M125AE" H 3090 1875 50  0001 C CNN "manf#"
@@
 F 0 "J1" H 2705 6257 50  0000 C CNN
 F 1 "USB_B_Micro" H 2705 6166 50  0000 C CNN
-F 2 "Connect:USB_Micro-B_10103594-0001LF" H 2800 5740 50  0001 C CNN
+F 2 "Connector_USB:USB_Micro-B_Amphenol_10103594-0001LF_Horizontal" H 2800 5740 50  0001 C CNN
 F 3 "~" H 2800 5740 50  0001 C CNN
 F 4 "629105150521" H 2650 5790 50  0001 C CNN "manf#"
@@
 F 0 "J2" H 1305 5897 50  0000 C CNN
 F 1 "SWD programmer" H 1305 5806 50  0000 C CNN
-F 2 "Pines:62000421121" H 1255 5680 50  0001 C CNN
+F 2 "Connector_PinHeader_1.00mm:PinHeader_2x02_P1.00mm_Vertical_SMD" H 1255 5680 50  0001 C CNN
 F 3 "~" H 1255 5680 50  0001 C CNN
 	1    1255 5680
@@
 F 0 "D3" V 5436 6861 50  0000 R CNN
 F 1 "D_Schottky" H 5375 6850 50  0000 R CNN
-F 2 "Diodes_SMD:D_SOD-123" H 5390 6940 50  0001 C CNN
+F 2 "Diode_SMD:D_SOD-123" H 5390 6940 50  0001 C CNN
 F 3 "~" H 5390 6940 50  0001 C CNN
 F 4 "STPS1L60ZFY" V 5390 6940 50  0001 C CNN "manf#"
@@
 F 0 "D2" V 5340 6840 50  0000 R CNN
 F 1 "D_Schottky" H 5325 6945 50  0000 R CNN
-F 2 "Diodes_SMD:D_SOD-123" H 5245 6850 50  0001 C CNN
+F 2 "Diode_SMD:D_SOD-123" H 5245 6850 50  0001 C CNN
 F 3 "~" H 5245 6850 50  0001 C CNN
 F 4 "STPS1L60ZFY" V 5245 6850 50  0001 C CNN "manf#"
@@
 F 0 "C5" H 3480 2595 50  0000 L CNN
 F 1 "0.1uF" H 3380 2430 50  0000 L CNN
-F 2 "Capacitors_SMD:C_0805_HandSoldering" H 3600 2510 50  0001 C CNN
+F 2 "Capacitor_SMD:C_0805_2012Metric_Pad1.15x1.40mm_HandSolder" H 3600 2510 50  0001 C CNN
 F 3 "~" H 3600 2510 50  0001 C CNN
 F 4 "08051C104J4T4A" H 3600 2510 50  0001 C CNN "manf#"
@@
 F 0 "C6" H 3897 2556 50  0000 L CNN
 F 1 "0.1uF" H 3835 2415 50  0000 L CNN
-F 2 "Capacitors_SMD:C_0805_HandSoldering" H 3805 2510 50  0001 C CNN
+F 2 "Capacitor_SMD:C_0805_2012Metric_Pad1.15x1.40mm_HandSolder" H 3805 2510 50  0001 C CNN
 F 3 "~" H 3805 2510 50  0001 C CNN
 F 4 "08051C104J4T4A" H 3805 2510 50  0001 C CNN "manf#"
@@
 F 0 "J3" H 7130 5867 50  0000 C CNN
 F 1 "ESP32-Exp" H 7130 5776 50  0000 C CNN
-F 2 "Pines:610X1221821" H 7080 5450 50  0001 C CNN
+F 2 "Connector_PinHeader_1.00mm:PinHeader_2x06_P1.00mm_Vertical_SMD" H 7080 5450 50  0001 C CNN
 F 3 "~" H 7080 5450 50  0001 C CNN
 F 4 "ESP32" H 7080 5450 50  0001 C CNN "manf#"
@@
 F 0 "R6" H 6689 5026 50  0000 L CNN
 F 1 "10K" H 6689 4935 50  0000 L CNN
-F 2 "Resistors_SMD:R_0805_HandSoldering" H 6630 4980 50  0001 C CNN
+F 2 "Resistor_SMD:R_0805_2012Metric_Pad1.15x1.40mm_HandSolder" H 6630 4980 50  0001 C CNN
 F 3 "~" H 6630 4980 50  0001 C CNN
 F 4 "CRCW080510K0FKEAC" H 6630 4980 50  0001 C CNN "manf#"
@@
 F 0 "R7" H 8224 5926 50  0000 L CNN
 F 1 "10K" H 8224 5835 50  0000 L CNN
-F 2 "Resistors_SMD:R_0805_HandSoldering" H 8165 5880 50  0001 C CNN
+F 2 "Resistor_SMD:R_0805_2012Metric_Pad1.15x1.40mm_HandSolder" H 8165 5880 50  0001 C CNN
 F 3 "~" H 8165 5880 50  0001 C CNN
 F 4 "CRCW080510K0FKEAC" H 8165 5880 50  0001 C CNN "manf#"
@@
 F 0 "U2" H 2120 4772 50  0000 C CNN
 F 1 "ATSAMD21G18A-AU" H 2120 4681 50  0000 C CNN
-F 2 "Housings_QFP:TQFP-48_7x7mm_Pitch0.5mm" H 2120 2905 50  0001 L BNN
+F 2 "Package_QFP:TQFP-48_7x7mm_P0.5mm" H 2120 2905 50  0001 L BNN
 F 3 "3.01 USD" H 2120 2905 50  0001 L BNN
 F 4 "Microchip" H 2120 2905 50  0001 L BNN "Campo4"
